Commit message: solve collisions
The collision were not working.

File: urdf/f1_robot.urdf (robot description, URDF)
Before this commit: robot f1_robot, 7 links, 6 joints
Links:
- removed link base_footprint
- removed link front_right_wheel
- removed link imu_link
- removed link rear_left_wheel
- removed link rear_right_wheel
Joints:
- removed joint base_joint
- removed joint front_right_wheel_joint
- removed joint imu_joint
- removed joint rear_left_wheel_joint
- removed joint rear_right_wheel_joint
- joint front_left_wheel_joint: origin xyz=${wheel_xoff_front} ${base_width/2 + wheel_width/2} ${-wheel_zoff} rpy=1.5708 0 0 -> xyz=${wheel_xoff_front} ${base_width/2 + wheel_width/2} ${-wheel_zoff} rpy=0 0 0

Commit message: Robot generated in gz & rviz
collision, joints and links are stable

File: urdf/f1_robot.urdf (robot description, URDF)
Before this commit: robot f1_robot, 2 links, 1 joints
Links:
- added link base_footprint
- added link front_right_wheel; collision cylinder length=${wheel_width} radius=${wheel_radius}; visual cylinder length=${wheel_width} radius=${wheel_radius}
- added link rear_left_wheel; collision cylinder length=${wheel_width} radius=${wheel_radius}; visual cylinder length=${wheel_width} radius=${wheel_radius}
- added link rear_right_wheel; collision cylinder length=${wheel_width} radius=${wheel_radius}; visual cylinder length=${wheel_width} radius=${wheel_radius}
Joints:
- added joint base_joint: type fixed, parent base_link, child base_footprint, origin xyz=0.0 0.0 ${-(wheel_radius+wheel_zoff)} rpy=0 0 0
- added joint front_right_wheel_joint: type revolute, parent base_link, child front_right_wheel, origin xyz=${wheel_xoff_front} ${-base_width/2 - wheel_width/2} ${-wheel_zoff} rpy=0 0 0, axis 0 1 0, limit lower=-1 upper=1 effort=1000 velocity=1
- added joint rear_left_wheel_joint: type continuous, parent base_link, child rear_left_wheel, origin xyz=${wheel_xoff_rear} ${base_width/2 + wheel_width/2} ${-wheel_zoff} rpy=0 0 0, axis 0 1 0
- added joint rear_right_wheel_joint: type continuous, parent base_link, child rear_right_wheel, origin xyz=${wheel_xoff_rear} ${-base_width/2 - wheel_width/2} ${-wheel_zoff} rpy=0 0 0, axis 0 1 0

Commit message: Hokuyo laser scanner added

File: urdf/f1_robot.urdf (robot description, URDF)
Before this commit: robot f1_robot, 7 links, 6 joints
Links:
- link lidar_link: geometry collision box size=0.1 0.1 0.1; visual mesh filename=file://$(find f1_robot_model)//meshes/hokuyo.stl

Commit message: f1 tenth added

File: urdf/f1_robot.urdf (robot description, URDF)
Before this commit: robot f1_robot, 7 links, 6 joints
Links:
- link front_left_wheel: mass None -> 1.3729096e+00
- link front_right_wheel: mass None -> 1.3729096e+00
- link lidar_link: geometry collision box size=0.1 0.1 0.1; visual mesh filename=file://$(find f1_robot_model)/meshes/hokuyo.stl
- link rear_left_wheel: mass None -> 1.3729096e+00
- link rear_right_wheel: mass None -> 1.3729096e+00
Joints:
- removed joint front_left_wheel_joint
- removed joint front_right_wheel_joint
- removed joint rear_left_wheel_joint
- removed joint rear_right_wheel_joint
- added joint front_left_joint: type revolute, parent base_link, child front_left_wheel, origin xyz=${wheel_xoff_front} ${base_width/2 + wheel_width/2} ${-wheel_zoff} rpy=0 0 0, axis 0 1 0, limit lower=-1 upper=1 effort=1000 velocity=1
- added joint front_right_joint: type revolute, parent base_link, child front_right_wheel, origin xyz=${wheel_xoff_front} ${-base_width/2 - wheel_width/2} ${-wheel_zoff} rpy=0 0 0, axis 0 1 0, limit lower=-1 upper=1 effort=1000 velocity=1
- added joint rear_left_joint: type continuous, parent base_link, child rear_left_wheel, origin xyz=${wheel_xoff_rear} ${base_width/2 + wheel_width/2} ${-wheel_zoff} rpy=0 0 0, axis 0 1 0
- added joint rear_right_joint: type continuous, parent base_link, child rear_right_wheel, origin xyz=${wheel_xoff_rear} ${-base_width/2 - wheel_width/2} ${-wheel_zoff} rpy=0 0 0, axis 0 1 0
