Commit message: added the space of the car appear

File: urdf/racecar.urdf (robot description, URDF)
Before this commit: robot racecar, 10 links, 9 joints
Links:
- removed link chassis_inertia
Joints:
- removed joint chassis_inertia_joint

Commit message: base footplrint link added

File: urdf/racecar.urdf (robot description, URDF)
Before this commit: robot racecar, 9 links, 8 joints
Links:
- added link base_footprint
Joints:
- added joint base_joint: type fixed, parent base_link, child base_footprint, origin xyz=0.0 0.0 -0.05 rpy=0 0 0
- joint base_link_joint: origin xyz=0 0 0.05 rpy=0 0 0 -> xyz=0 0 0 rpy=0 0 0

Commit message: updated

File: urdf/racecar.urdf (robot description, URDF)
Before this commit: robot racecar, 10 links, 9 joints
Joints:
- joint base_link_joint: origin xyz=0 0 0 rpy=0 0 0 -> xyz=-0.16 0 0 rpy=0 0 0
